File: hardware/USBAudioBridge.kicad_sch (KiCad schematic)
At the start: 0 parts

Commit message: Post first draft design review complete
Changed lines of the file:
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@@
 		)
 	)
-	(text "DESIGN NOTES\nPower: USB VBUS (PTC fused) -> AP7361C 3.3 V main rail; LP5907 3.3 V low-noise rail (+3V3_CLK) for the audio clock.\n  RT1010 internal DC-DC (4.7 uH) generates the 1.1 V VDD_SOC rail. VDD_SNVS_IN is tied to 3.3 V (no backup battery).\n  Arty PMOD VCC (pins 6/12) is NOT connected to 3.3 V: JP601 is an open solder jumper. Grounds are common.\nClocks: 24.000 MHz crystal (system/USB PLL), 32.768 kHz crystal (RTC), 24.576 MHz XO (audio master) -> CDCV304 1:4 buffer:\n  Y0 -> GPIO_08 SAI1_MCLK (input, GPR1 SAI1_MCLK_DIR=0, SAI1_MCLK1_SEL=011)\n  Y1 -> GPIO_AD_03 GPT2_CLK (counts MCLK between USB SOFs for the async feedback endpoint; needs ipg_clk >= 98.4 MHz)\n  Y2 -> PMOD JB9 MCLK to the FPGA.  RT1010 SAI1 is I2S clock master for both buses.\nBoot: BOOT_MODE[1:0]=10 (internal boot, FlexSPI-A QSPI NOR) by default. Hold BOOT and press RESET for 01 (serial downloader over USB).\nDebug: MCU-Link 10-pin Cortex debug header (SWD + SWO), 3-pin LPUART1 console header.\n\nPIN MAP\n  GPIO_01..03  SAI1 RX BCLK/SYNC/DATA0   (I2S input bus, FPGA -> RT1010)\n  GPIO_04,06,07 SAI1 TX DATA0/BCLK/SYNC  (I2S output bus, RT1010 -> FPGA)\n  GPIO_05      SAI1 TX/RX DATA1 (aux)    GPIO_08  SAI1_MCLK in\n  GPIO_09/10   LPUART1 RX/TX             GPIO_11/12  LED1/LED2\n  GPIO_AD_04/05/06 LPSPI1 SDO/PCS0/SCK   GPIO_SD_05  LPSPI1 SDI (daisy select 1)\n  GPIO_AD_00 PMOD_INT, AD_07 PMOD_RST, AD_01/02 PMOD_GPIO0/1 (LPI2C2 or LPUART4 capable)\n  GPIO_AD_09..13 SWO/TDI/JTAG_MOD/SWCLK/SWDIO\n  GPIO_SD_06..11 FlexSPI-A QSPI flash    GPIO_SD_00..04 BT_CFG / BOOT_MODE straps"
+	(text "DESIGN NOTES\nPower: USB VBUS (PTC fused) -> AP7361C 3.3 V main rail; LP5907 3.3 V low-noise rail (+3V3_CLK) for the audio clock.\n  RT1010 internal DC-DC (4.7 uH) generates the 1.1 V VDD_SOC rail. VDD_SNVS_IN is tied to 3.3 V (no backup battery).\n  Arty PMOD VCC (pins 6/12) is NOT connected to 3.3 V: JP601 is an open solder jumper. Grounds are common.\nClocks: 24.000 MHz crystal (system/USB PLL), 32.768 kHz crystal (RTC), 24.576 MHz XO (audio master, Epson SG-210STF) -> CDCV304 1:4 buffer:\n  Y0 -> GPIO_08 SAI1_MCLK (input, GPR1 SAI1_MCLK_DIR=0, SAI1_MCLK1_SEL=011)\n  Y1 -> GPIO_AD_03 GPT2_CLK (counts MCLK between USB SOFs for the async feedback endpoint; needs ipg_clk >= 98.4 MHz)\n  Y2/Y3 -> PMOD JB1/JB7, the MCLK pin of each I2S row.  RT1010 SAI1 is I2S clock master for both buses.\nPMOD JB matches the Digilent Pmod I2S2: top row (1-4) MCLK/LRCK/SCLK/SDIN carries FPGA -> RT1010 audio, bottom row (7-10) MCLK/LRCK/SCLK/SDOUT carries RT1010 -> FPGA audio.\nBoot: BOOT_MODE[1:0]=10 (internal boot, FlexSPI-A QSPI NOR) by default. Hold BOOT and press RESET for 01 (serial downloader over USB).\nDebug: MCU-Link 10-pin Cortex debug header (SWD + SWO), 3-pin LPUART1 console header.\n\nPIN MAP\n  GPIO_01..03  SAI1 RX BCLK/SYNC/DATA0   (I2S input bus, FPGA -> RT1010)\n  GPIO_04,06,07 SAI1 TX DATA0/BCLK/SYNC  (I2S output bus, RT1010 -> FPGA)\n  GPIO_08      SAI1_MCLK in              GPIO_00, 05, 13, AD_08, AD_14  spare (NC)\n  GPIO_09/10   LPUART1 RX/TX             GPIO_11/12  LED1/LED2\n  GPIO_AD_04/05/06 LPSPI1 SDO/PCS0/SCK   GPIO_SD_05  LPSPI1 SDI (daisy select 1)\n  GPIO_AD_00 PMOD_INT, AD_07 PMOD_RST, AD_01/02 PMOD_GPIO0/1 (LPI2C2 or LPUART4 capable)\n  GPIO_AD_09..13 SWO/TDI/JTAG_MOD/SWCLK/SWDIO\n  GPIO_SD_06..11 FlexSPI-A QSPI flash    GPIO_SD_00..04 BT_CFG / BOOT_MODE straps"
 		(exclude_from_sim no)
 		(at 30.48 152.4 0)

Commit message: finished pcb layout. reviewing
Parts:
- added H1, H2: MountingHole_M3, MountingHole:MountingHole_3.2mm_M3, symbol Mechanical:MountingHole
Other:
- note added: "H1, H2: M3 holes for a standoff that takes USB cable strain off the PMOD headers."
- note added: "NXP i.MX RT1010 USB 2.0 HS asynchronous audio device bridging to an Arty A7 FPGA board over two PMOD ports (JB: SPI + GPIO, JC: I2S)."
- note removed: "NXP i.MX RT1010 USB 2.0 HS asynchronous audio device bridging to an Arty A7 FPGA board over two PMOD ports (JB: I2S, JC: SPI + GPIO)."
Changed lines of the file:
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@@
 		)
 	)
-	(text "DESIGN NOTES\nPower: USB VBUS (PTC fused) -> AP7361C 3.3 V main rail; LP5907 3.3 V low-noise rail (+3V3_CLK) for the audio clock.\n  RT1010 internal DC-DC (4.7 uH) generates the 1.1 V VDD_SOC rail. VDD_SNVS_IN is tied to 3.3 V (no backup battery).\n  Arty PMOD VCC (pins 6/12) is NOT connected to 3.3 V: JP601 is an open solder jumper. Grounds are common.\nClocks: 24.000 MHz crystal (system/USB PLL), 32.768 kHz crystal (RTC), 24.576 MHz XO (audio master, Epson SG-210STF) -> CDCV304 1:4 buffer:\n  Y0 -> GPIO_08 SAI1_MCLK (input, GPR1 SAI1_MCLK_DIR=0, SAI1_MCLK1_SEL=011)\n  Y1 -> GPIO_AD_03 GPT2_CLK (counts MCLK between USB SOFs for the async feedback endpoint; needs ipg_clk >= 98.4 MHz)\n  Y2/Y3 -> PMOD JB1/JB7, the MCLK pin of each I2S row.  RT1010 SAI1 is I2S clock master for both buses.\nPMOD JB matches the Digilent Pmod I2S2: top row (1-4) MCLK/LRCK/SCLK/SDIN carries FPGA -> RT1010 audio, bottom row (7-10) MCLK/LRCK/SCLK/SDOUT carries RT1010 -> FPGA audio.\nBoot: BOOT_MODE[1:0]=10 (internal boot, FlexSPI-A QSPI NOR) by default. Hold BOOT and press RESET for 01 (serial downloader over USB).\nDebug: MCU-Link 10-pin Cortex debug header (SWD + SWO), 3-pin LPUART1 console header.\n\nPIN MAP\n  GPIO_01..03  SAI1 RX BCLK/SYNC/DATA0   (I2S input bus, FPGA -> RT1010)\n  GPIO_04,06,07 SAI1 TX DATA0/BCLK/SYNC  (I2S output bus, RT1010 -> FPGA)\n  GPIO_08      SAI1_MCLK in              GPIO_00, 05, 13, AD_08, AD_14  spare (NC)\n  GPIO_09/10   LPUART1 RX/TX             GPIO_11/12  LED1/LED2\n  GPIO_AD_04/05/06 LPSPI1 SDO/PCS0/SCK   GPIO_SD_05  LPSPI1 SDI (daisy select 1)\n  GPIO_AD_00 PMOD_INT, AD_07 PMOD_RST, AD_01/02 PMOD_GPIO0/1 (LPI2C2 or LPUART4 capable)\n  GPIO_AD_09..13 SWO/TDI/JTAG_MOD/SWCLK/SWDIO\n  GPIO_SD_06..11 FlexSPI-A QSPI flash    GPIO_SD_00..04 BT_CFG / BOOT_MODE straps"
+	(text "DESIGN NOTES\nPower: USB VBUS (PTC fused) -> AP7361C 3.3 V main rail; LP5907 3.3 V low-noise rail (+3V3_CLK) for the audio clock.\n  RT1010 internal DC-DC (4.7 uH) generates the 1.1 V VDD_SOC rail. VDD_SNVS_IN is tied to 3.3 V (no backup battery).\n  Arty PMOD VCC (pins 6/12) is NOT connected to 3.3 V: JP601 is an open solder jumper. Grounds are common.\nClocks: 24.000 MHz crystal (system/USB PLL), 32.768 kHz crystal (RTC), 24.576 MHz XO (audio master, Epson SG-210STF) -> CDCV304 1:4 buffer:\n  Y0 -> GPIO_08 SAI1_MCLK (input, GPR1 SAI1_MCLK_DIR=0, SAI1_MCLK1_SEL=011)\n  Y1 -> GPIO_AD_03 GPT2_CLK (counts MCLK between USB SOFs for the async feedback endpoint; needs ipg_clk >= 98.4 MHz)\n  Y2/Y3 -> PMOD JC1/JC7, the MCLK pin of each I2S row.  RT1010 SAI1 is I2S clock master for both buses.\nPMOD JC matches the Digilent Pmod I2S2: top row (1-4) MCLK/LRCK/SCLK/SDIN carries FPGA -> RT1010 audio, bottom row (7-10) MCLK/LRCK/SCLK/SDOUT carries RT1010 -> FPGA audio.\nBoot: BOOT_MODE[1:0]=10 (internal boot, FlexSPI-A QSPI NOR) by default. Hold BOOT and press RESET for 01 (serial downloader over USB).\nDebug: MCU-Link 10-pin Cortex debug header (SWD + SWO), 3-pin LPUART1 console header.\n\nPIN MAP\n  GPIO_01..03  SAI1 RX BCLK/SYNC/DATA0   (I2S input bus, FPGA -> RT1010)\n  GPIO_04,06,07 SAI1 TX DATA0/BCLK/SYNC  (I2S output bus, RT1010 -> FPGA)\n  GPIO_08      SAI1_MCLK in              GPIO_00, 05, 13, AD_08, AD_14  spare (NC)\n  GPIO_09/10   LPUART1 RX/TX             GPIO_11/12  LED1/LED2\n  GPIO_AD_04/05/06 LPSPI1 SDO/PCS0/SCK   GPIO_SD_05  LPSPI1 SDI (daisy select 1)\n  GPIO_AD_00 PMOD_INT, AD_07 PMOD_RST, AD_01/02 PMOD_GPIO0/1 (LPI2C2 or LPUART4 capable)\n  GPIO_AD_09..13 SWO/TDI/JTAG_MOD/SWCLK/SWDIO\n  GPIO_SD_06..11 FlexSPI-A QSPI flash    GPIO_SD_00..04 BT_CFG / BOOT_MODE straps"
 		(exclude_from_sim no)
 		(at 30.48 152.4 0)
@@
 		)
 	)
-	(text "NXP i.MX RT1010 USB 2.0 HS asynchronous audio device bridging to an Arty A7 FPGA board over two PMOD ports (JB: I2S, JC: SPI + GPIO)."
+	(text "H1, H2: M3 holes for a standoff that takes USB cable strain\noff the PMOD headers."
+		(exclude_from_sim no)
+		(at 205.74 73.66 0)
+		(effects
+			(font
+				(size 1.27 1.27)
+			)
+			(justify left)
+		)
+	)
+	(text "NXP i.MX RT1010 USB 2.0 HS asynchronous audio device bridging to an Arty A7 FPGA board over two PMOD ports (JB: SPI + GPIO, JC: I2S)."
 		(exclude_from_sim no)
 		(at 30.48 38.1 0)
@@
 		)
 	)
+	(symbol
+		(lib_id "Mechanical:MountingHole")
+		(at 228.6 63.5 0)
+		(unit 1)
+		(body_style 1)
+		(exclude_from_sim no)
+		(in_bom no)
+		(on_board yes)
+		(in_pos_files yes)
+		(dnp no)
+		(property "Reference" "H2"
+			(at 228.6 58.42 0)
+			(show_name no)
+			(do_not_autoplace no)
+			(effects
+				(font
+					(size 1.27 1.27)
+				)
+			)
+		)
+		(property "Value" "MountingHole_M3"
+			(at 228.6 60.96 0)
+			(show_name no)
+			(do_not_autoplace no)
+			(effects
+				(font
+					(size 1.27 1.27)
+				)
+			)
+		)
+		(property "Footprint" "MountingHole:MountingHole_3.2mm_M3"
+			(at 228.6 63.5 0)
+			(hide yes)
+			(show_name no)
+			(do_not_autoplace no)
+			(effects
+				(font
+					(size 1.27 1.27)
+				)
+			)
+		)
+		(property "Datasheet" ""
+			(at 228.6 63.5 0)
+			(hide yes)
+			(show_name no)
+			(do_not_autoplace no)
+			(effects
+				(font
+					(size 1.27 1.27)
+				)
+			)
+		)
+		(property "Description" "Mounting Hole without connection"
+			(at 228.6 63.5 0)
+			(hide yes)
+			(show_name no)
+			(do_not_autoplace no)
+			(effects
+				(font
+					(size 1.27 1.27)
+				)
+			)
+		)
+		(instances)
+	)
+	(symbol
+		(lib_id "Mechanical:MountingHole")
+		(at 215.9 63.5 0)
+		(unit 1)
+		(body_style 1)
+		(exclude_from_sim no)
+		(in_bom no)
+		(on_board yes)
+		(in_pos_files yes)
+		(dnp no)
+		(property "Reference" "H1"
+			(at 215.9 58.42 0)
+			(show_name no)
+			(do_not_autoplace no)
+			(effects
+				(font
+					(size 1.27 1.27)
+				)
+			)
+		)
+		(property "Value" "MountingHole_M3"
+			(at 215.9 60.96 0)
+			(show_name no)
+			(do_not_autoplace no)
+			(effects
+				(font
+					(size 1.27 1.27)
+				)
+			)
+		)
+		(property "Footprint" "MountingHole:MountingHole_3.2mm_M3"
+			(at 215.9 63.5 0)
+			(hide yes)
+			(show_name no)
+			(do_not_autoplace no)
+			(effects
+				(font
+					(size 1.27 1.27)
+				)
+			)
+		)
+		(property "Datasheet" ""
+			(at 215.9 63.5 0)
+			(hide yes)
+			(show_name no)
+			(do_not_autoplace no)
+			(effects
+				(font
+					(size 1.27 1.27)
+				)
+			)
+		)
+		(property "Description" "Mounting Hole without connection"
+			(at 215.9 63.5 0)
+			(hide yes)
+			(show_name no)
+			(do_not_autoplace no)
+			(effects
+				(font
+					(size 1.27 1.27)
+				)
+			)
+		)
+		(instances)
+	)
 	(sheet

Commit message: post pcb layout design review
Other:
- note added: "NXP i.MX RT1010 USB 2.0 HS asynchronous audio device bridging to an Arty A7 FPGA board over two PMOD ports (JB: I2S, JC: SPI + GPIO)."
- note removed: "NXP i.MX RT1010 USB 2.0 HS asynchronous audio device bridging to an Arty A7 FPGA board over two PMOD ports (JB: SPI + GPIO, JC: I2S)."
Changed lines of the file:
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@@
 		)
 	)
-	(text "DESIGN NOTES\nPower: USB VBUS (PTC fused) -> AP7361C 3.3 V main rail; LP5907 3.3 V low-noise rail (+3V3_CLK) for the audio clock.\n  RT1010 internal DC-DC (4.7 uH) generates the 1.1 V VDD_SOC rail. VDD_SNVS_IN is tied to 3.3 V (no backup battery).\n  Arty PMOD VCC (pins 6/12) is NOT connected to 3.3 V: JP601 is an open solder jumper. Grounds are common.\nClocks: 24.000 MHz crystal (system/USB PLL), 32.768 kHz crystal (RTC), 24.576 MHz XO (audio master, Epson SG-210STF) -> CDCV304 1:4 buffer:\n  Y0 -> GPIO_08 SAI1_MCLK (input, GPR1 SAI1_MCLK_DIR=0, SAI1_MCLK1_SEL=011)\n  Y1 -> GPIO_AD_03 GPT2_CLK (counts MCLK between USB SOFs for the async feedback endpoint; needs ipg_clk >= 98.4 MHz)\n  Y2/Y3 -> PMOD JC1/JC7, the MCLK pin of each I2S row.  RT1010 SAI1 is I2S clock master for both buses.\nPMOD JC matches the Digilent Pmod I2S2: top row (1-4) MCLK/LRCK/SCLK/SDIN carries FPGA -> RT1010 audio, bottom row (7-10) MCLK/LRCK/SCLK/SDOUT carries RT1010 -> FPGA audio.\nBoot: BOOT_MODE[1:0]=10 (internal boot, FlexSPI-A QSPI NOR) by default. Hold BOOT and press RESET for 01 (serial downloader over USB).\nDebug: MCU-Link 10-pin Cortex debug header (SWD + SWO), 3-pin LPUART1 console header.\n\nPIN MAP\n  GPIO_01..03  SAI1 RX BCLK/SYNC/DATA0   (I2S input bus, FPGA -> RT1010)\n  GPIO_04,06,07 SAI1 TX DATA0/BCLK/SYNC  (I2S output bus, RT1010 -> FPGA)\n  GPIO_08      SAI1_MCLK in              GPIO_00, 05, 13, AD_08, AD_14  spare (NC)\n  GPIO_09/10   LPUART1 RX/TX             GPIO_11/12  LED1/LED2\n  GPIO_AD_04/05/06 LPSPI1 SDO/PCS0/SCK   GPIO_SD_05  LPSPI1 SDI (daisy select 1)\n  GPIO_AD_00 PMOD_INT, AD_07 PMOD_RST, AD_01/02 PMOD_GPIO0/1 (LPI2C2 or LPUART4 capable)\n  GPIO_AD_09..13 SWO/TDI/JTAG_MOD/SWCLK/SWDIO\n  GPIO_SD_06..11 FlexSPI-A QSPI flash    GPIO_SD_00..04 BT_CFG / BOOT_MODE straps"
+	(text "DESIGN NOTES\nPower: USB VBUS (PTC fused) -> AP7361C 3.3 V main rail; LP5907 3.3 V low-noise rail (+3V3_CLK) for the audio clock.\n  RT1010 internal DC-DC (4.7 uH) generates the 1.1 V VDD_SOC rail. VDD_SNVS_IN is tied to 3.3 V (no backup battery).\n  Arty PMOD VCC (pins 6/12) is NOT connected to 3.3 V: JP601 is an open solder jumper. Grounds are common.\nClocks: 24.000 MHz crystal (system/USB PLL), 32.768 kHz crystal (RTC), 24.576 MHz XO (audio master, Epson SG-210STF) -> CDCV304 1:4 buffer:\n  Y0 -> GPIO_08 SAI1_MCLK (input, GPR1 SAI1_MCLK_DIR=0, SAI1_MCLK1_SEL=011)\n  Y1 -> GPIO_AD_03 GPT2_CLK (counts MCLK between USB SOFs for the async feedback endpoint; needs ipg_clk >= 98.4 MHz)\n  Y2/Y3 -> PMOD JB1/JB7, the MCLK pin of each I2S row.  RT1010 SAI1 is I2S clock master for both buses.\nPMOD JB matches the Digilent Pmod I2S2 (JB1/JB3 are Artix-7 clock-capable pins): top row (1-4) MCLK/LRCK/SCLK/SDIN carries FPGA -> RT1010 audio, bottom row (7-10) MCLK/LRCK/SCLK/SDOUT carries RT1010 -> FPGA audio.\nBoot: BOOT_MODE[1:0]=10 (internal boot, FlexSPI-A QSPI NOR) by default. Hold BOOT and press RESET for 01 (serial downloader over USB).\nDebug: MCU-Link 10-pin Cortex debug header (SWD + SWO), 3-pin LPUART1 console header.\n\nPIN MAP\n  GPIO_01..03  SAI1 RX BCLK/SYNC/DATA0   (I2S input bus, FPGA -> RT1010)\n  GPIO_04,06,07 SAI1 TX DATA0/BCLK/SYNC  (I2S output bus, RT1010 -> FPGA)\n  GPIO_08      SAI1_MCLK in              GPIO_00, 05, 13, AD_08, AD_14  spare (NC)\n  GPIO_09/10   LPUART1 RX/TX             GPIO_11/12  LED1/LED2\n  GPIO_AD_04/05/06 LPSPI1 SDO/PCS0/SCK   GPIO_SD_05  LPSPI1 SDI (daisy select 1)\n  GPIO_AD_00 PMOD_INT, AD_07 PMOD_RST, AD_01/02 PMOD_GPIO0/1 (LPI2C2 or LPUART4 capable)\n  GPIO_AD_09..13 SWO/TDI/JTAG_MOD/SWCLK/SWDIO\n  GPIO_SD_06..11 FlexSPI-A QSPI flash    GPIO_SD_00..04 BT_CFG / BOOT_MODE straps"
 		(exclude_from_sim no)
 		(at 30.48 152.4 0)
@@
 		)
 	)
-	(text "NXP i.MX RT1010 USB 2.0 HS asynchronous audio device bridging to an Arty A7 FPGA board over two PMOD ports (JB: SPI + GPIO, JC: I2S)."
+	(text "NXP i.MX RT1010 USB 2.0 HS asynchronous audio device bridging to an Arty A7 FPGA board over two PMOD ports (JB: I2S, JC: SPI + GPIO)."
 		(exclude_from_sim no)
 		(at 30.48 38.1 0)
