File: hardware/audio_pmod.kicad_sch (KiCad schematic)
At the start: 26 parts, among them J601 PMOD_JB, J602 PMOD_JC, U601 CDCV304PW, X601 24.576MHz

Commit message: Post first draft design review complete
Parts:
- removed X601: 24.576MHz, Oscillator:Oscillator_SMD_ECS_2520MV-xxx-xx-4Pin_2.5x2.0mm, symbol Oscillator:ECS-2520MV-xxx-xx
- added X601: 24.576MHz, Oscillator:Oscillator_SMD_SeikoEpson_SG210-4Pin_2.5x2.0mm, symbol Oscillator:SG-210STF
Connections:
- net I2S_AUX_DATA is gone; now on net I2S_TX_DATA: R611.2
- net JB_AUX_DATA is gone; now on net JB_TX_DATA: J601.10 (Pin_10), R611.1
- net +3V3_CLK: now also X601.1 (~{ST}), X601.4 (Vcc)
- net GND: now also X601.2 (GND)
- net I2S_RX_BCLK: now also R607.1; no longer R609.2
- net I2S_RX_DATA: now also R608.1; no longer R606.1
- net I2S_RX_LRCLK: now also R606.1; no longer R610.2
- net I2S_TX_BCLK: now also R610.2; no longer R608.1
- net I2S_TX_DATA: no longer R607.1
- net I2S_TX_LRCLK: now also R609.2; no longer R605.1
- net JB_RX_BCLK: now also J601.3 (Pin_3), R607.2; no longer J601.7 (Pin_7), R609.1
- net JB_RX_DATA: now also J601.4 (Pin_4), R608.2; no longer J601.2 (Pin_2), R606.2
- net JB_RX_LRCLK: now also J601.2 (Pin_2), R606.2; no longer J601.8 (Pin_8), R610.1
- net JB_TX_BCLK: now also J601.9 (Pin_9), R610.1; no longer J601.4 (Pin_4), R608.2
- net JB_TX_DATA: no longer J601.3 (Pin_3), R607.2
- net JB_TX_LRCLK: now also J601.8 (Pin_8), R609.1; no longer J601.1 (Pin_1), R605.2
- net at R601.1: now also X601.3 (OUT)
- net at U601.8 (1Y3): now also R605.1
- net JB_MCLK renamed JB_RX_MCLK
- net JB_RX_MCLK: now also J601.1 (Pin_1); no longer J601.9 (Pin_9)
- new net JB_TX_MCLK: J601.7 (Pin_7), R605.2
- no-connect marks 1 -> 0
Other:
- note added: "PMOD JB (Arty high-speed port): I2S, Pmod I2S2 pinout"
- note added: "Pmod I2S2 pinout (host = FPGA): 1-4 D/A row: MCLK, LRCK, SCLK, SDIN = FPGA -> RT1010 (SAI1 RX) 7-10 A/D row: MCLK, LRCK, SCLK, SDOUT = RT1010 -> FPGA (SAI1 TX) All clocks are driven by this board: the FPGA must treat JB1-3 and JB7-9 as inputs. Arty HS pairs 1-2 and 7-8 couple MCLK with LRCK (LRCK is a slow, sampled signal)."
- note added: "Series terminations at the buffer outputs. Y0 -> RT1010 SAI1_MCLK (GPIO_08) Y1 -> RT1010 GPT2_CLK (GPIO_AD_03), async feedback Y2 -> PMOD JB1 (MCLK, top row) Y3 -> PMOD JB7 (MCLK, bottom row)"
- note removed: "PMOD JB (Arty high-speed port): I2S"
- note removed: "Pins 1-4 + 9 follow PMOD Type 7 (LRCLK, DAC data in, ADC data out, BCLK, MCLK) for the RT1010 TX clocks. RX bus clocks on 7/8, aux SAI1 data line on 10. Arty HS pairs: 1-2, 3-4, 7-8, 9-10 (MCLK paired with the quiet aux line)."
- note removed: "Series terminations at the buffer outputs. Y0 -> RT1010 SAI1_MCLK (GPIO_08) Y1 -> RT1010 GPT2_CLK (GPIO_AD_03), async feedback Y2 -> FPGA via PMOD JB9"

Commit message: finished pcb layout. reviewing
Parts:
- J601, J602: footprint Connector_PinHeader_2.54mm:PinHeader_2x06_P2.54mm_Horizontal -> USBAudioBridge:PMOD_Peripheral_2x06_P2.54mm_Horizontal
- JP601: now left out of the parts list
Connections:
- net I2S_RX_BCLK: now also R615.1; no longer R607.1
- net I2S_RX_DATA: now also R616.1; no longer R608.1
- net I2S_RX_LRCLK: now also R614.1; no longer R606.1
- net I2S_TX_BCLK: now also R618.2; no longer R610.2
- net I2S_TX_DATA: now also R619.2; no longer R611.2
- net I2S_TX_LRCLK: now also R617.2; no longer R609.2
- net PMOD_GPIO0: now also R612.2; no longer R618.2
- net PMOD_GPIO1: now also R613.2; no longer R619.2
- net PMOD_INT: now also R610.2; no longer R616.2
- net PMOD_RST: now also R611.2; no longer R617.2
- net SPI_CS: now also R606.1; no longer R612.1
- net SPI_MISO: now also R608.1; no longer R614.1
- net SPI_MOSI: now also R607.1; no longer R613.1
- net SPI_SCK: now also R609.1; no longer R615.1
- net JB_RX_BCLK renamed JB_SPI_MISO
- net JB_SPI_MISO: now also R608.2; no longer R607.2
- net JB_RX_DATA renamed JB_SPI_SCK
- net JB_SPI_SCK: now also R609.2; no longer R608.2
- net JB_RX_LRCLK renamed JB_SPI_CS
- net JB_SPI_CS: now also J601.1 (Pin_1); no longer J601.2 (Pin_2)
- net JB_RX_MCLK renamed JC_RX_MCLK
- net JC_RX_MCLK: now also J602.1 (Pin_1); no longer J601.1 (Pin_1)
- net JB_TX_BCLK renamed JB_GPIO0
- net JB_GPIO0: now also R612.1; no longer R610.1
- net JB_TX_DATA renamed JB_GPIO1
- net JB_GPIO1: now also R613.1; no longer R611.1
- net JB_TX_LRCLK renamed JB_RST
- net JB_RST: now also R611.1; no longer R609.1
- net JB_TX_MCLK renamed JB_INT
- net JB_INT: now also R610.1; no longer R605.2
- net JC_GPIO0 renamed JC_TX_BCLK
- net JC_GPIO1 renamed JC_TX_DATA
- net JC_INT renamed JC_TX_MCLK
- net JC_TX_MCLK: now also R605.2; no longer R616.1
- net JC_RST renamed JC_TX_LRCLK
- removed net JC_SPI_CS: J602.1 (Pin_1), R612.2
- net JC_SPI_MISO renamed JC_RX_BCLK
- net JC_RX_BCLK: now also R615.2; no longer R614.2
- net JC_SPI_MOSI renamed JC_RX_LRCLK
- net JC_RX_LRCLK: now also R614.2; no longer R613.2
- net JC_SPI_SCK renamed JC_RX_DATA
- net JC_RX_DATA: now also R616.2; no longer R615.2
- new net JB_SPI_MOSI: J601.2 (Pin_2), R607.2
Other:
- note added: "PMOD JB (Arty high-speed port): SPI + GPIO"
- note added: "PMOD JC (Arty high-speed port): I2S, Pmod I2S2 pinout"
- note added: "Pmod I2S2 pinout (host = FPGA): 1-4 D/A row: MCLK, LRCK, SCLK, SDIN = FPGA -> RT1010 (SAI1 RX) 7-10 A/D row: MCLK, LRCK, SCLK, SDOUT = RT1010 -> FPGA (SAI1 TX) All clocks are driven by this board: the FPGA must treat JC1-3 and JC7-9 as inputs. Arty HS pairs 1-2 and 7-8 couple MCLK with LRCK (LRCK is a slow, sampled signal)."
- note added: "Series terminations at the buffer outputs. Y0 -> RT1010 SAI1_MCLK (GPIO_08) Y1 -> RT1010 GPT2_CLK (GPIO_AD_03), async feedback Y2 -> PMOD JC1 (MCLK, top row) Y3 -> PMOD JC7 (MCLK, bottom row)"
- note removed: "PMOD JB (Arty high-speed port): I2S, Pmod I2S2 pinout"
- note removed: "PMOD JC (Arty high-speed port): SPI + GPIO"
- note removed: "Pmod I2S2 pinout (host = FPGA): 1-4 D/A row: MCLK, LRCK, SCLK, SDIN = FPGA -> RT1010 (SAI1 RX) 7-10 A/D row: MCLK, LRCK, SCLK, SDOUT = RT1010 -> FPGA (SAI1 TX) All clocks are driven by this board: the FPGA must treat JB1-3 and JB7-9 as inputs. Arty HS pairs 1-2 and 7-8 couple MCLK with LRCK (LRCK is a slow, sampled signal)."
- note removed: "Series terminations at the buffer outputs. Y0 -> RT1010 SAI1_MCLK (GPIO_08) Y1 -> RT1010 GPT2_CLK (GPIO_AD_03), async feedback Y2 -> PMOD JB1 (MCLK, top row) Y3 -> PMOD JB7 (MCLK, bottom row)"

Commit message: post pcb layout design review
Connections:
- net I2S_RX_BCLK: now also R607.1; no longer R615.1
- net I2S_RX_DATA: now also R608.1; no longer R616.1
- net I2S_RX_LRCLK: now also R606.1; no longer R614.1
- net I2S_TX_BCLK: now also R610.2; no longer R618.2
- net I2S_TX_DATA: now also R611.2; no longer R619.2
- net I2S_TX_LRCLK: now also R609.2; no longer R617.2
- net PMOD_GPIO0: now also R618.2; no longer R612.2
- net PMOD_GPIO1: now also R619.2; no longer R613.2
- net PMOD_INT: now also R616.2; no longer R610.2
- net PMOD_RST: now also R617.2; no longer R611.2
- net SPI_CS: now also R612.1; no longer R606.1
- net SPI_MISO: now also R614.1; no longer R608.1
- net SPI_MOSI: now also R613.1; no longer R607.1
- net SPI_SCK: now also R615.1; no longer R609.1
- net JB_GPIO0 renamed JB_TX_BCLK
- net JB_TX_BCLK: now also R610.1; no longer R612.1
- net JB_GPIO1 renamed JB_TX_DATA
- net JB_TX_DATA: now also R611.1; no longer R613.1
- net JB_INT renamed JB_TX_MCLK
- net JB_TX_MCLK: now also R605.2; no longer R610.1
- net JB_RST renamed JB_TX_LRCLK
- net JB_TX_LRCLK: now also R609.1; no longer R611.1
- net JB_SPI_CS renamed JB_RX_LRCLK
- net JB_RX_LRCLK: now also J601.2 (Pin_2); no longer J601.1 (Pin_1)
- net JB_SPI_MISO renamed JB_RX_BCLK
- net JB_RX_BCLK: now also R607.2; no longer R608.2
- removed net JB_SPI_MOSI: J601.2 (Pin_2), R607.2
- net JB_SPI_SCK renamed JB_RX_DATA
- net JB_RX_DATA: now also R608.2; no longer R609.2
- net JC_RX_BCLK renamed JC_SPI_MISO
- net JC_SPI_MISO: now also R614.2; no longer R615.2
- net JC_RX_DATA renamed JC_SPI_SCK
- net JC_SPI_SCK: now also R615.2; no longer R616.2
- net JC_RX_LRCLK renamed JC_SPI_MOSI
- net JC_SPI_MOSI: now also R613.2; no longer R614.2
- net JC_RX_MCLK renamed JB_RX_MCLK
- net JB_RX_MCLK: now also J601.1 (Pin_1); no longer J602.1 (Pin_1)
- net JC_TX_BCLK renamed JC_GPIO0
- net JC_TX_DATA renamed JC_GPIO1
- net JC_TX_LRCLK renamed JC_RST
- net JC_TX_MCLK renamed JC_INT
- net JC_INT: now also R616.1; no longer R605.2
- new net JC_SPI_CS: J602.1 (Pin_1), R612.2
Other:
- note added: "PMOD JB (Arty high-speed port): I2S, Pmod I2S2 pinout"
- note added: "PMOD JC (Arty high-speed port): SPI + GPIO"
- note added: "Pmod I2S2 pinout (host = FPGA): 1-4 D/A row: MCLK, LRCK, SCLK, SDIN = FPGA -> RT1010 (SAI1 RX) 7-10 A/D row: MCLK, LRCK, SCLK, SDOUT = RT1010 -> FPGA (SAI1 TX) All clocks are driven by this board: the FPGA must treat JB1-3 and JB7-9 as inputs. JB1 (MCLK) and JB3 (SCLK) land on Artix-7 clock-capable pins E15 (SRCC) and D15 (MRCC); run SAI1 TX synchronous to RX so JB3 clocks both directions."
- note added: "Series terminations at the buffer outputs. Y0 -> RT1010 SAI1_MCLK (GPIO_08) Y1 -> RT1010 GPT2_CLK (GPIO_AD_03), async feedback Y2 -> PMOD JB1 (MCLK, top row) Y3 -> PMOD JB7 (MCLK, bottom row)"
- note removed: "PMOD JB (Arty high-speed port): SPI + GPIO"
- note removed: "PMOD JC (Arty high-speed port): I2S, Pmod I2S2 pinout"
- note removed: "Pmod I2S2 pinout (host = FPGA): 1-4 D/A row: MCLK, LRCK, SCLK, SDIN = FPGA -> RT1010 (SAI1 RX) 7-10 A/D row: MCLK, LRCK, SCLK, SDOUT = RT1010 -> FPGA (SAI1 TX) All clocks are driven by this board: the FPGA must treat JC1-3 and JC7-9 as inputs. Arty HS pairs 1-2 and 7-8 couple MCLK with LRCK (LRCK is a slow, sampled signal)."
- note removed: "Series terminations at the buffer outputs. Y0 -> RT1010 SAI1_MCLK (GPIO_08) Y1 -> RT1010 GPT2_CLK (GPIO_AD_03), async feedback Y2 -> PMOD JC1 (MCLK, top row) Y3 -> PMOD JC7 (MCLK, bottom row)"

Commit message: Add fab pipeline, sourcing, CI and developer reference manual
- tools/fab.py: ERC/DRC gate, then JLCPCB (LCSC BOM, rotation-corrected
  CPL) and PCBWay (MPN BOM, centroid) packages with Gerbers, drill,
  assembly drawings, schematic PDF and order notes
- .github/workflows/fab.yml: runs fab.py in kicad/kicad:10.0.7; artifacts
  on push/PR, release assets on v* tags
- design.py: MPN/Manufacturer/LCSC for every BOM line (checked against
  JLCPCB stock); SG-210SCBA oscillator, Liming 200 uW 24 MHz crystal,
  PTS810SJG switches, USB4105-GF-A-120, ~2 V LEDs
- R603 DNP: GPT2 cannot count 24.576 MHz (external clock < PERCLK/4,
  PERCLK <= 75 MHz); async feedback comes from SAI sample counts
- Via drill 0.3 -> 0.2 mm (pads unchanged) for PCBWay's 5 mil ring
- Drill/place origin at the board's lower-left corner; legible Fab refs
- pcb.py --sync-fields updates fields/DNP without re-routing
- docs/reference-manual.md: RT1010 firmware and Arty A7 reference
Parts:
- C601, C602: LCSC (none) -> C1525; MPN (none) -> CL05B104KO5NNNC; Manufacturer (none) -> Samsung Electro-Mechanics
- J601, J602: LCSC (none) -> C492434; MPN (none) -> PZ254R-12-12P; Manufacturer (none) -> XFCN
- R601: LCSC (none) -> C25092; MPN (none) -> 0402WGF220JTCE; Manufacturer (none) -> UNI-ROYAL
- R602, R604, R605, R606, R607, R608, R609, R610, R611, R612, R613, R614, R615, R616, R617, R618, R619: LCSC (none) -> C25105; MPN (none) -> 0402WGF330JTCE; Manufacturer (none) -> UNI-ROYAL
- R603: LCSC (none) -> C25105; MPN (none) -> 0402WGF330JTCE; Manufacturer (none) -> UNI-ROYAL; now not fitted
- U601: LCSC (none) -> C105237
- X601: LCSC (none) -> C5154204; MPN SG-210STF 24.5760ML -> X1G004591A052; Manufacturer Epson -> Seiko Epson; Spec 24.576 MHz CMOS SPXO, 1.62-3.63 V, +/-50 ppm, -40..85 C, 2.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 -> SG-210SCBA 24.576000 MHz L: CMOS SPXO, 2.7-3.6 V, +/-50 ppm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
Other:
- note added: "Series terminations at the buffer outputs. Y0 -> RT1010 SAI1_MCLK (GPIO_08) Y1 -> R603 (DNP) -> GPIO_AD_03 GPT2_CLK, spare Y2 -> PMOD JB1 (MCLK, top row) Y3 -> PMOD JB7 (MCLK, bottom row)"
- note removed: "Series terminations at the buffer outputs. Y0 -> RT1010 SAI1_MCLK (GPIO_08) Y1 -> RT1010 GPT2_CLK (GPIO_AD_03), async feedback Y2 -> PMOD JB1 (MCLK, top row) Y3 -> PMOD JB7 (MCLK, bottom row)"
