File: hardware/boot_flash.kicad_sch (KiCad schematic)
At the start: 16 parts, among them Q401 BSS84, SW401 BOOT, U1 MIMXRT1011DAE5A, U401 W25Q128JVSIQ

Commit message: Add fab pipeline, sourcing, CI and developer reference manual
- tools/fab.py: ERC/DRC gate, then JLCPCB (LCSC BOM, rotation-corrected
  CPL) and PCBWay (MPN BOM, centroid) packages with Gerbers, drill,
  assembly drawings, schematic PDF and order notes
- .github/workflows/fab.yml: runs fab.py in kicad/kicad:10.0.7; artifacts
  on push/PR, release assets on v* tags
- design.py: MPN/Manufacturer/LCSC for every BOM line (checked against
  JLCPCB stock); SG-210SCBA oscillator, Liming 200 uW 24 MHz crystal,
  PTS810SJG switches, USB4105-GF-A-120, ~2 V LEDs
- R603 DNP: GPT2 cannot count 24.576 MHz (external clock < PERCLK/4,
  PERCLK <= 75 MHz); async feedback comes from SAI sample counts
- Via drill 0.3 -> 0.2 mm (pads unchanged) for PCBWay's 5 mil ring
- Drill/place origin at the board's lower-left corner; legible Fab refs
- pcb.py --sync-fields updates fields/DNP without re-routing
- docs/reference-manual.md: RT1010 firmware and Arty A7 reference
Parts:
- C401: LCSC (none) -> C1525; MPN (none) -> CL05B104KO5NNNC; Manufacturer (none) -> Samsung Electro-Mechanics
- C402: LCSC (none) -> C52923; MPN (none) -> CL05A105KA5NQNC; Manufacturer (none) -> Samsung Electro-Mechanics
- Q401: LCSC (none) -> C82079; MPN BSS84 -> BSS84LT1G; Manufacturer (none) -> onsemi
- R401, R402, R403, R404, R407, R408, R409, R410: LCSC (none) -> C25744; MPN (none) -> 0402WGF1002TCE; Manufacturer (none) -> UNI-ROYAL
- R405, R406: LCSC (none) -> C11702; MPN (none) -> 0402WGF1001TCE; Manufacturer (none) -> UNI-ROYAL
- SW401: LCSC (none) -> C221895; MPN PTS810SJM250SMTRLFS -> PTS810SJG250SMTRLFS
- U1: LCSC (none) -> C1575810; MPN (none) -> MIMXRT1011DAE5A; Manufacturer (none) -> NXP
- U401: LCSC (none) -> C97521
