File: hardware/mcu_io.kicad_sch (KiCad schematic)
At the start: 11 parts, among them J501 SWD, J502 UART, U1 MIMXRT1011DAE5A

Commit message: Post first draft design review complete
Connections:
- net I2S_AUX_DATA: no longer names the net of U1.8 (GPIO_05)
- no-connect marks 5 -> 6
Changed lines of the file:
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@@
+	)
+	(no_connect
+		(at 149.86 99.06)
 	)
 	(no_connect
@@
 	(wire
 		(pts
-			(xy 149.86 99.06) (xy 147.32 99.06)
-		)
-		(stroke
-			(width 0)
-			(type default)
-		)
-	)
-	(wire
-		(pts
 			(xy 180.34 93.98) (xy 182.88 93.98)
 		)
@@
 			(hide yes)
 			(show_name no)
-			(do_not_autoplace no)
-			(effects
-				(font
-					(size 1.27 1.27)
-				)
-			)
-		)
-	)
-	(global_label "I2S_AUX_DATA"
-		(shape bidirectional)
-		(at 147.32 99.06 180)
-		(fields_autoplaced yes)
-		(effects
-			(font
-				(size 1.27 1.27)
-			)
-			(justify right)
-		)
-		(property "Intersheetrefs" "${INTERSHEET_REFS}"
-			(at 147.32 99.06 0)
-			(hide yes)
-			(show_name no)

Commit message: post pcb layout design review
Parts:
- J501: footprint Connector_PinHeader_1.27mm:PinHeader_2x05_P1.27mm_Vertical_SMD -> USBAudioBridge:Samtec_FTSH-105-01-L-DV-K; MPN (none) -> FTSH-105-01-L-DV-K; Manufacturer (none) -> Samtec; Spec 2x5 1.27 mm SMD header (Samtec FTSH-105-01-L-DV-K or eq.) -> 2x5 1.27 mm SMD header with keying shroud (Cortex debug)
Other:
- note added: "MCU-Link debug (10-pin Cortex, 1.27 mm, keyed)"
- note removed: "MCU-Link debug (10-pin Cortex, 1.27 mm)"
Changed lines of the file:
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@@
 		)
 	)
-	(text "MCU-Link debug (10-pin Cortex, 1.27 mm)"
+	(text "MCU-Link debug (10-pin Cortex, 1.27 mm, keyed)"
 		(exclude_from_sim no)
 		(at 275.59 27.94 0)
@@
 			)
 		)
-		(property "Footprint" "Connector_PinHeader_1.27mm:PinHeader_2x05_P1.27mm_Vertical_SMD"
+		(property "Footprint" "USBAudioBridge:Samtec_FTSH-105-01-L-DV-K"
 			(at 325.12 63.5 0)
 			(hide yes)
@@
 			)
 		)
-		(property "Spec" "2x5 1.27 mm SMD header (Samtec FTSH-105-01-L-DV-K or eq.)"
+		(property "MPN" "FTSH-105-01-L-DV-K"
+			(at 325.12 63.5 0)
+			(hide yes)
+			(show_name no)
+			(do_not_autoplace no)
+			(effects
+				(font
+					(size 1.27 1.27)
+				)
+			)
+		)
+		(property "Manufacturer" "Samtec"
+			(at 325.12 63.5 0)
+			(hide yes)
+			(show_name no)
+			(do_not_autoplace no)
+			(effects
+				(font
+					(size 1.27 1.27)
+				)
+			)
+		)
+		(property "Spec" "2x5 1.27 mm SMD header with keying shroud (Cortex debug)"
 			(at 325.12 63.5 0)
 			(hide yes)

Commit message: Add fab pipeline, sourcing, CI and developer reference manual
- tools/fab.py: ERC/DRC gate, then JLCPCB (LCSC BOM, rotation-corrected
  CPL) and PCBWay (MPN BOM, centroid) packages with Gerbers, drill,
  assembly drawings, schematic PDF and order notes
- .github/workflows/fab.yml: runs fab.py in kicad/kicad:10.0.7; artifacts
  on push/PR, release assets on v* tags
- design.py: MPN/Manufacturer/LCSC for every BOM line (checked against
  JLCPCB stock); SG-210SCBA oscillator, Liming 200 uW 24 MHz crystal,
  PTS810SJG switches, USB4105-GF-A-120, ~2 V LEDs
- R603 DNP: GPT2 cannot count 24.576 MHz (external clock < PERCLK/4,
  PERCLK <= 75 MHz); async feedback comes from SAI sample counts
- Via drill 0.3 -> 0.2 mm (pads unchanged) for PCBWay's 5 mil ring
- Drill/place origin at the board's lower-left corner; legible Fab refs
- pcb.py --sync-fields updates fields/DNP without re-routing
- docs/reference-manual.md: RT1010 firmware and Arty A7 reference
Parts:
- D501: LCSC (none) -> C2289; MPN (none) -> KT-0603YG; Manufacturer (none) -> Hubei KENTO
- D502: LCSC (none) -> C2287; MPN (none) -> KT-0603Y; Manufacturer (none) -> Hubei KENTO
- J501: LCSC (none) -> C5155080
- J502: LCSC (none) -> C2937625; MPN (none) -> PZ254V-11-03P; Manufacturer (none) -> XFCN
- R501, R503, R504: LCSC (none) -> C25744; MPN (none) -> 0402WGF1002TCE; Manufacturer (none) -> UNI-ROYAL
- R502: LCSC (none) -> C25900; MPN (none) -> 0402WGF4701TCE; Manufacturer (none) -> UNI-ROYAL
- R505, R506: LCSC (none) -> C11702; MPN (none) -> 0402WGF1001TCE; Manufacturer (none) -> UNI-ROYAL
- U1: LCSC (none) -> C1575810; MPN (none) -> MIMXRT1011DAE5A; Manufacturer (none) -> NXP
