File: hardware/mcu_power.kicad_sch (KiCad schematic)
At the start: 33 parts, among them U1 MIMXRT1011DAE5A

Commit message: Add fab pipeline, sourcing, CI and developer reference manual
- tools/fab.py: ERC/DRC gate, then JLCPCB (LCSC BOM, rotation-corrected
  CPL) and PCBWay (MPN BOM, centroid) packages with Gerbers, drill,
  assembly drawings, schematic PDF and order notes
- .github/workflows/fab.yml: runs fab.py in kicad/kicad:10.0.7; artifacts
  on push/PR, release assets on v* tags
- design.py: MPN/Manufacturer/LCSC for every BOM line (checked against
  JLCPCB stock); SG-210SCBA oscillator, Liming 200 uW 24 MHz crystal,
  PTS810SJG switches, USB4105-GF-A-120, ~2 V LEDs
- R603 DNP: GPT2 cannot count 24.576 MHz (external clock < PERCLK/4,
  PERCLK <= 75 MHz); async feedback comes from SAI sample counts
- Via drill 0.3 -> 0.2 mm (pads unchanged) for PCBWay's 5 mil ring
- Drill/place origin at the board's lower-left corner; legible Fab refs
- pcb.py --sync-fields updates fields/DNP without re-routing
- docs/reference-manual.md: RT1010 firmware and Arty A7 reference
Parts:
- C201: LCSC (none) -> C45783; MPN (none) -> CL21A226MAQNNNE; Manufacturer (none) -> Samsung Electro-Mechanics
- C202, C205, C206, C207, C210, C211, C212, C214, C216, C217, C218, C219, C223: LCSC (none) -> C16772; MPN (none) -> CL05B224KO5NNNC; Manufacturer (none) -> Samsung Electro-Mechanics
- C203, C204, C209, C213, C215, C228, C229, C230: LCSC (none) -> C23733; MPN (none) -> CL05A475MP5NRNC; Manufacturer (none) -> Samsung Electro-Mechanics
- C208, C220: LCSC (none) -> C19702; MPN (none) -> CL10A106KP8NNNC; Manufacturer (none) -> Samsung Electro-Mechanics
- C221, C224, C225, C226, C227: LCSC (none) -> C1525; MPN (none) -> CL05B104KO5NNNC; Manufacturer (none) -> Samsung Electro-Mechanics
- C222: LCSC (none) -> C52923; MPN (none) -> CL05A105KA5NQNC; Manufacturer (none) -> Samsung Electro-Mechanics
- L201: LCSC (none) -> C780206
- R201: LCSC (none) -> C25776; MPN (none) -> 0402WGF3002TCE; Manufacturer (none) -> UNI-ROYAL
- U1: LCSC (none) -> C1575810; MPN (none) -> MIMXRT1011DAE5A; Manufacturer (none) -> NXP
