File: hardware/mcu_system.kicad_sch (KiCad schematic)
At the start: 14 parts, among them SW301 RESET, U1 MIMXRT1011DAE5A, U301 MCP120T-300I/TT, Y301 24MHz, Y302 32.768kHz

Commit message: Post first draft design review complete
Parts:
- U301: Spec open-drain, Vtrip 2.93 V (> 2.6 V DCDC_IN UVLO) -> open-drain, Vtrip 2.925 V (> 2.6 V DCDC_IN UVLO)
Changed lines of the file:
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@@
 			)
 		)
-		(property "Spec" "open-drain, Vtrip 2.93 V (> 2.6 V DCDC_IN UVLO)"
+		(property "Spec" "open-drain, Vtrip 2.925 V (> 2.6 V DCDC_IN UVLO)"
 			(at 299.72 66.04 0)
 			(hide yes)

Commit message: Add fab pipeline, sourcing, CI and developer reference manual
- tools/fab.py: ERC/DRC gate, then JLCPCB (LCSC BOM, rotation-corrected
  CPL) and PCBWay (MPN BOM, centroid) packages with Gerbers, drill,
  assembly drawings, schematic PDF and order notes
- .github/workflows/fab.yml: runs fab.py in kicad/kicad:10.0.7; artifacts
  on push/PR, release assets on v* tags
- design.py: MPN/Manufacturer/LCSC for every BOM line (checked against
  JLCPCB stock); SG-210SCBA oscillator, Liming 200 uW 24 MHz crystal,
  PTS810SJG switches, USB4105-GF-A-120, ~2 V LEDs
- R603 DNP: GPT2 cannot count 24.576 MHz (external clock < PERCLK/4,
  PERCLK <= 75 MHz); async feedback comes from SAI sample counts
- Via drill 0.3 -> 0.2 mm (pads unchanged) for PCBWay's 5 mil ring
- Drill/place origin at the board's lower-left corner; legible Fab refs
- pcb.py --sync-fields updates fields/DNP without re-routing
- docs/reference-manual.md: RT1010 firmware and Arty A7 reference
Parts:
- C301: LCSC (none) -> C15849; MPN (none) -> CL10A105KB8NNNC; Manufacturer (none) -> Samsung Electro-Mechanics
- C302, C303, C304, C305: LCSC (none) -> C32949; MPN (none) -> CL05C100JB5NNNC; Manufacturer (none) -> Samsung Electro-Mechanics
- C306, C307: LCSC (none) -> C1525; MPN (none) -> CL05B104KO5NNNC; Manufacturer (none) -> Samsung Electro-Mechanics
- R301: LCSC (none) -> C11490; MPN (none) -> 0402WGF2204TCE; Manufacturer (none) -> UNI-ROYAL; Spec 5% 0402 -> 1% 0402
- R302: LCSC (none) -> C25744; MPN (none) -> 0402WGF1002TCE; Manufacturer (none) -> UNI-ROYAL
- SW301: LCSC (none) -> C221895; MPN PTS810SJM250SMTRLFS -> PTS810SJG250SMTRLFS
- U1: LCSC (none) -> C1575810; MPN (none) -> MIMXRT1011DAE5A; Manufacturer (none) -> NXP
- U301: LCSC (none) -> C625180
- Y301: LCSC (none) -> C2981672; MPN (none) -> 3225-24-8-10-10/A; Manufacturer (none) -> Suzhou Liming; Spec 24.000 MHz fundamental, CL 8 pF, ESR <= 80 ohm, drive >= 25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 -> 24.000 MHz fundamental, CL 8 pF, ESR <= 60 ohm, rated drive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
- Y302: LCSC (none) -> C48615; MPN (none) -> Q13FC13500002; Manufacturer (none) -> Seiko Epson
