File: hardware/power_usb.kicad_sch (KiCad schematic)
At the start: 21 parts, among them J101 USB_C_Receptacle, U101 USBLC6-2SC6, U102 AP7361C-33E, U103 LP5907MFX-3.3

Commit message: Post first draft design review complete
Other:
- note added: "ESD: place U101 at the connector, route D+/D- through its pads (flow-through). 90 ohm differential pair. No series resistors: the RT1010 HS PHY has calibrated on-die 45 ohm terminations (RM 36.3.5.1)."
- note removed: "ESD: place U101 at the connector, route D+/D- through its pads (flow-through). 90 ohm differential pair."
Changed lines of the file:
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@@
-		)
-	)
-	(text "ESD: place U101 at the connector,\nroute D+/D- through its pads (flow-through).\n90 ohm differential pair."
-		(exclude_from_sim no)
-		(at 119.38 86.36 0)
-		(effects
-			(font
-				(size 1.27 1.27)
-			)
-			(justify left)
 		)
 	)
@@
 		(effects
 			(font
+				(size 1.27 1.27)
+			)
+			(justify left)
+		)
+	)
+	(text "ESD: place U101 at the connector,\nroute D+/D- through its pads (flow-through).\n90 ohm differential pair.\nNo series resistors: the RT1010 HS PHY has\ncalibrated on-die 45 ohm terminations (RM 36.3.5.1)."
+		(exclude_from_sim no)
+		(at 104.14 86.36 0)
+		(effects
+			(font

Commit message: finished pcb layout. reviewing
Parts:
- TP101, TP102, TP103, TP104: now left out of the parts list

Commit message: Add fab pipeline, sourcing, CI and developer reference manual
- tools/fab.py: ERC/DRC gate, then JLCPCB (LCSC BOM, rotation-corrected
  CPL) and PCBWay (MPN BOM, centroid) packages with Gerbers, drill,
  assembly drawings, schematic PDF and order notes
- .github/workflows/fab.yml: runs fab.py in kicad/kicad:10.0.7; artifacts
  on push/PR, release assets on v* tags
- design.py: MPN/Manufacturer/LCSC for every BOM line (checked against
  JLCPCB stock); SG-210SCBA oscillator, Liming 200 uW 24 MHz crystal,
  PTS810SJG switches, USB4105-GF-A-120, ~2 V LEDs
- R603 DNP: GPT2 cannot count 24.576 MHz (external clock < PERCLK/4,
  PERCLK <= 75 MHz); async feedback comes from SAI sample counts
- Via drill 0.3 -> 0.2 mm (pads unchanged) for PCBWay's 5 mil ring
- Drill/place origin at the board's lower-left corner; legible Fab refs
- pcb.py --sync-fields updates fields/DNP without re-routing
- docs/reference-manual.md: RT1010 firmware and Arty A7 reference
Parts:
- C101: LCSC (none) -> C1538; MPN (none) -> 0402B472K500NT; Manufacturer (none) -> FH (Guangdong Fenghua)
- C102: LCSC (none) -> C19666; MPN (none) -> CL10A475KO8NNNC; Manufacturer (none) -> Samsung Electro-Mechanics
- C103, C104, C107: LCSC (none) -> C15849; MPN (none) -> CL10A105KB8NNNC; Manufacturer (none) -> Samsung Electro-Mechanics
- C105: LCSC (none) -> C19702; MPN (none) -> CL10A106KP8NNNC; Manufacturer (none) -> Samsung Electro-Mechanics
- C106: LCSC (none) -> C1525; MPN (none) -> CL05B104KO5NNNC; Manufacturer (none) -> Samsung Electro-Mechanics
- D101: LCSC (none) -> C2289; MPN (none) -> KT-0603YG; Manufacturer (none) -> Hubei KENTO
- F101: LCSC (none) -> C43379; MPN (none) -> SMD1206P050TF/13.2; Manufacturer (none) -> RUILON
- J101: LCSC (none) -> C5184243; MPN USB4105-GF-A -> USB4105-GF-A-120; Spec (none) -> -120: 1.20 mm shell stakes
- R101, R102: LCSC (none) -> C25905; MPN (none) -> 0402WGF5101TCE; Manufacturer (none) -> UNI-ROYAL
- R103: LCSC (none) -> C26083; MPN (none) -> 0402WGF1004TCE; Manufacturer (none) -> UNI-ROYAL; Spec 5% 0402 -> 1% 0402
- R104: LCSC (none) -> C11702; MPN (none) -> 0402WGF1001TCE; Manufacturer (none) -> UNI-ROYAL
- U101: LCSC (none) -> C7519
- U102: LCSC (none) -> C500795
- U103: LCSC (none) -> C80670
